File: PCB/Rev A/source/Cube OS/Cube OS.kicad_pcb (KiCad board)
At the start: 4 copper layers, 60 x 60 mm, 81 parts, among them J1 1S 3.7 V LiPo, J2 KH-TYPE-C-16P, M1 Motor_Servo, M2 Motor_Servo, Q1 AO3400A, SW1 JS202011JAQN, SW2 SPPJ320600, SW3 RESET, SW4 BOOT, U1 ESP32-S3-WROOM-1-N8R2, U10 Right Display, U11 Display, U12 Left Display, U13 MAX98357AETE+T, U14 TPS63802DLAR, U16 TPS7A0212PDBVR, U2 SHT45-AD1B-R2_Temp_Hu, U3 VEML7700-TT_SHORT, U4 LDLN025J28R, U5 ISM330DHCXTR_GYRO, U7 TCA6408ARGTR, U8 BQ24074RGTR_Batt, U9 Front Display

Commit message: Revert "Update Rev A PCB production package"
This reverts commit 683648053a19518fab4d864910172dd1a356c20e.
Parts:
- removed C10: 4.7uF, Capacitor_SMD:C_0402_1005Metric
- removed C11: 47uF, Capacitor_SMD:C_0805_2012Metric
- removed C7, C8, C9: 1 uF, Capacitor_SMD:C_0402_1005Metric
- removed R15, R20, R21, R22, R24: 10 kΩ, Resistor_SMD:R_0402_1005Metric
- removed R17, R18, R19, R23: 10Ω, Resistor_SMD:R_0603_1608Metric
- removed SW3: RESET, Cube_OS_Footprint:SW_TS-1088_XNP
- removed SW4: BOOT, Cube_OS_Footprint:SW_TS-1088_XNP
- removed TP1: GND, TestPoint:TestPoint_Pad_1.0x1.0mm
- removed TP10: CHG_PGOOD, TestPoint:TestPoint_Pad_1.0x1.0mm
- removed TP11: CHG_STAT, TestPoint:TestPoint_Pad_1.0x1.0mm
- removed TP12: DISP_SCLK, TestPoint:TestPoint_Pad_1.0x1.0mm
- removed TP13: DISP_MOSI, TestPoint:TestPoint_Pad_1.0x1.0mm
- removed TP14: DISP_BL_PWM, TestPoint:TestPoint_Pad_1.0x1.0mm
- removed TP2: USB_VBUS, TestPoint:TestPoint_Pad_1.0x1.0mm
- removed TP3: BAT_IN, TestPoint:TestPoint_Pad_1.0x1.0mm
- removed TP4: ESP32_EN, TestPoint:TestPoint_Pad_1.0x1.0mm
- removed TP5: Buck_IN, TestPoint:TestPoint_Pad_1.0x1.0mm
- removed TP6: Buck_OUT_3.3V, TestPoint:TestPoint_Pad_1.0x1.0mm
- removed TP7: ESP32_BOOT, TestPoint:TestPoint_Pad_1.0x1.0mm
- removed TP8: I2C_SDA, TestPoint:TestPoint_Pad_1.0x1.0mm
- removed TP9: I2C_SCL, TestPoint:TestPoint_Pad_1.0x1.0mm
- removed U11: Display, Cube_OS_Footprint:CON_5034801200_MOL
- removed U4: LDLN025J28R, Cube_OS_Footprint:FLIPCHIP4_0P658X0P658_STM
- added U15: LDLN025M25R, Cube_OS_Footprint:SOT23_DBV_TEX, F.Cu at (141.6, 133.6)
- R6: value 3.9kΩ -> 2.4 kΩ
- U1: value ESP32-S3-WROOM-1-N8R2 -> ESP32-S3-WROOM-1-N8R8
- U10, U12, U9: footprint Cube_OS_Footprint:CON_5034801200_MOL -> Cube_OS_Footprint:CONN_FH35C-15S-0.3SHW50_HIR
- U7: value TCA6408ARGTR -> Top Display; footprint Cube_OS_Footprint:RGT16_1P45X1P45 -> Cube_OS_Footprint:CONN_FH35C-15S-0.3SHW50_HIR
- moved SW1 60.2 mm to (125.0, 101.7)
- moved M1 56.0 mm to (108.0, 102.5)
- moved J1 46.3 mm to (151.0, 105.0)
- moved SW2 44.8 mm to (143.2, 105.0)
- moved R16 40.5 mm to (134.0, 114.5)
- moved TH1 30.4 mm to (150.0, 112.0), turned to 0 degrees
- moved U7 22.8 mm to (119.2, 115.9), turned to 0 degrees
- moved U5 5.14 mm to (136.3, 156.2)
- moved R12 0.31 mm to (152.0, 113.0), turned to 0 degrees
- turned U10 to -90 degrees
- turned U12 to 180 degrees
- turned U9 to 0 degrees
Connections:
- C2 pad 1: Net-(U14-VIN) -> Net-(U14-EN)
- J1 pad 1: GND -> Net-(J1-Pin_1)
- J1 pad 2: +BAT -> GND
- R12 pad 1: 3.3V -> Net-(U1-IO39)
- R13 pad 1: 3.3V -> Net-(U1-IO38)
- R16 pad 2: Net-(U7-P2) -> Net-(U1-IO5)
- SW1 pad 2: Net-(U14-EN) -> Net-(J1-Pin_1)
- SW1 pad 5: Net-(U14-VIN) -> +BAT
- U1 pad 10: /CAM_HREF -> /IMU_INT1
- U1 pad 15: unconnected-(U1-IO3-Pad15) -> /CAM_HREF
- U1 pad 16: unconnected-(U1-IO46-Pad16) -> /CAM_D6
- U1 pad 26: unconnected-(U1-IO45-Pad26) -> /CAM_D5
- U1 pad 27: Net-(U1-IO0) -> /CAM_VSYNC
- U1 pad 3: Net-(U1-EN) -> 3.3V
- U1 pad 31: /CAM_D6 -> Net-(U1-IO38)
- U1 pad 32: /CAM_D5 -> Net-(U1-IO39)
- U1 pad 5: /CAM_VSYNC -> Net-(U1-IO5)
- U10 pad 1: LEDK -> 3.3V
- U10 pad 10: 3.3V -> /DISP_DC
- U10 pad 11: /DISP_RIGHT_CS -> /DISP_MOSI
- U10 pad 12: GND -> unconnected-(U10-TE-Pad12)
- U10 pad 2: Net-(U10-LEDA) -> LEDK
- U10 pad 3: GND -> 3.3V
- U10 pad 4: unconnected-(U10-SDO-Pad4) -> 3.3V
- U10 pad 5: /DISP_RST -> GND
- U10 pad 6: /DISP_MOSI -> GND
- U10 pad 7: /DISP_DC -> /DISP_RST
- U10 pad 8: /DISP_SCLK -> /DISP_RIGHT_CS
- U10 pad 9: 3.3V -> /DISP_SCLK
- U12 pad 1: LEDK -> 3.3V
- U12 pad 10: 3.3V -> /DISP_DC
- U12 pad 11: /DISP_LEFT_CS -> /DISP_MOSI
- U12 pad 12: GND -> unconnected-(U12-TE-Pad12)
- U12 pad 2: Net-(U12-LEDA) -> LEDK
- U12 pad 3: GND -> 3.3V
- U12 pad 4: unconnected-(U12-SDO-Pad4) -> 3.3V
- U12 pad 5: /DISP_RST -> GND
- U12 pad 6: /DISP_MOSI -> GND
- U12 pad 7: /DISP_DC -> /DISP_RST
- U12 pad 8: /DISP_SCLK -> /DISP_LEFT_CS
- U12 pad 9: 3.3V -> /DISP_SCLK
- U14 pad 10: Net-(U14-VIN) -> Net-(U14-EN)
- U2 pad 4: GND -> 3.3V
- U5 pad 4: unconnected-(U5-INT1-Pad4) -> /IMU_INT1
- U7 pad 1: Net-(U7-*RESET) -> 3.3V
- U7 pad 10: unconnected-(U7-P7-Pad10) -> /DISP_DC
- U7 pad 11: Net-(U7-*INT) -> /DISP_MOSI
- U7 pad 12: /I2C_SCL -> unconnected-(U7-TE-Pad12)
- U7 pad 13: /I2C_SDA -> GND
- U7 pad 14: 3.3V -> GND
- U7 pad 15: 3.3V -> GND
- U7 pad 2: /CHG_PGOOD -> LEDK
- U7 pad 3: /CHG_STAT -> 3.3V
- U7 pad 4: Net-(U7-P2) -> 3.3V
- U7 pad 5: unconnected-(U7-P3-Pad5) -> GND
- U7 pad 7: unconnected-(U7-P4-Pad7) -> /DISP_RST
- U7 pad 8: unconnected-(U7-P5-Pad8) -> /DISP_TOP_CS
- U7 pad 9: unconnected-(U7-P6-Pad9) -> /DISP_SCLK
- U8 pad 10: Net-(U14-VIN) -> Net-(U14-EN)
- U8 pad 11: Net-(U14-VIN) -> Net-(U14-EN)
- U9 pad 1: LEDK -> 3.3V
- U9 pad 10: 3.3V -> /DISP_DC
- U9 pad 11: /DISP_FRONT_CS -> /DISP_MOSI
- U9 pad 12: GND -> unconnected-(U9-TE-Pad12)
- U9 pad 2: Net-(U9-LEDA) -> LEDK
- U9 pad 3: GND -> 3.3V
- U9 pad 4: unconnected-(U9-SDO-Pad4) -> 3.3V
- U9 pad 5: /DISP_RST -> GND
- U9 pad 6: /DISP_MOSI -> GND
- U9 pad 7: /DISP_DC -> /DISP_RST
- U9 pad 8: /DISP_SCLK -> /DISP_FRONT_CS
- U9 pad 9: 3.3V -> /DISP_SCLK
Routing:
- net Net-(U1-IO5): track 0.00 -> 85.0 mm, vias 0 -> 2
- net Net-(U1-EN): track 79.2 -> 0.00 mm, vias 3 -> 0
- net Net-(U14-VIN): track 65.1 -> 0.00 mm, vias 4 -> 0
- net /CAM_VSYNC: track 66.3 -> 12.8 mm
- net /SERVO1_PWM: track 79.2 -> 29.5 mm, vias 4 -> 2
- net Net-(U7-P2): track 49.0 -> 0.00 mm, vias 2 -> 0
- net Net-(U1-IO0): track 48.7 -> 0.00 mm, vias 4 -> 0
- net Net-(U14-EN): track 54.2 -> 9.55 mm
- net Net-(U1-IO39): track 0.00 -> 41.0 mm, vias 0 -> 4
- net Net-(U1-IO38): track 0.00 -> 39.6 mm, vias 0 -> 4
- net GND: track 142.6 -> 103.7 mm, vias 193 -> 63
- net /CHG_PGOOD: track 39.0 -> 2.26 mm, vias 6 -> 0
- net Net-(U8-TS): track 36.2 -> 5.92 mm
- net Net-(J1-Pin_1): track 0.00 -> 29.9 mm
- net /I2C_SCL: track 73.5 -> 44.2 mm, vias 7 -> 5
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- removed copper zone on F.Cu, net (none)
Other:
- outline, holes or cut-outs redrawn
- board text removed: "+BAT"
- board text removed: "GND"

Commit message: Update Rev A hardware files
Parts:
- removed U15: LDLN025M25R, Cube_OS_Footprint:SOT23_DBV_TEX
- added C10: 4.7uF, Capacitor_SMD:C_0402_1005Metric, F.Cu at (151.8, 106.5)
- added C11: 47uF, Capacitor_SMD:C_0805_2012Metric, F.Cu at (153.2, 106.0)
- added C7: 1 uF, Capacitor_SMD:C_0402_1005Metric, F.Cu at (140.5, 137.5)
- added C8: 1 uF, Capacitor_SMD:C_0402_1005Metric, F.Cu at (128.0, 132.0)
- added C9: 1 uF, Capacitor_SMD:C_0402_1005Metric, F.Cu at (127.5, 135.5)
- added R15: 10 kΩ, Resistor_SMD:R_0402_1005Metric, F.Cu at (133.0, 107.0)
- added R17: 10Ω, Resistor_SMD:R_0603_1608Metric, F.Cu at (118.5, 113.6)
- added R18: 10Ω, Resistor_SMD:R_0603_1608Metric, F.Cu at (116.2, 158.5)
- added R19: 10Ω, Resistor_SMD:R_0603_1608Metric, F.Cu at (148.5, 134.8)
- added R20: 10 kΩ, Resistor_SMD:R_0402_1005Metric, F.Cu at (138.0, 121.0)
- added R21: 10 kΩ, Resistor_SMD:R_0402_1005Metric, F.Cu at (144.5, 123.5)
- added R22: 10 kΩ, Resistor_SMD:R_0402_1005Metric, F.Cu at (118.0, 123.0)
- added R23: 10Ω, Resistor_SMD:R_0603_1608Metric, F.Cu at (132.8, 113.4)
- added R24: 10 kΩ, Resistor_SMD:R_0402_1005Metric, F.Cu at (133.0, 103.0)
- added SW3: RESET, Cube_OS_Footprint:SW_TS-1088_XNP, F.Cu at (137.2, 107.0)
- added SW4: BOOT, Cube_OS_Footprint:SW_TS-1088_XNP, F.Cu at (137.2, 103.0)
- added TP1: GND, TestPoint:TestPoint_Pad_1.0x1.0mm, F.Cu at (158.0, 145.5)
- added TP10: CHG_PGOOD, TestPoint:TestPoint_Pad_1.0x1.0mm, F.Cu at (143.5, 110.5)
- added TP11: CHG_STAT, TestPoint:TestPoint_Pad_1.0x1.0mm, F.Cu at (145.5, 113.5)
- added TP12: DISP_SCLK, TestPoint:TestPoint_Pad_1.0x1.0mm, F.Cu at (152.2, 146.0)
- added TP13: DISP_MOSI, TestPoint:TestPoint_Pad_1.0x1.0mm, F.Cu at (149.5, 148.0)
- added TP14: DISP_BL_PWM, TestPoint:TestPoint_Pad_1.0x1.0mm, F.Cu at (140.5, 134.5)
- added TP2: USB_VBUS, TestPoint:TestPoint_Pad_1.0x1.0mm, F.Cu at (129.0, 148.5)
- added TP3: BAT_IN, TestPoint:TestPoint_Pad_1.0x1.0mm, F.Cu at (152.5, 152.5)
- added TP4: ESP32_EN, TestPoint:TestPoint_Pad_1.0x1.0mm, F.Cu at (117.0, 156.8)
- added TP5: Buck_IN, TestPoint:TestPoint_Pad_1.0x1.0mm, F.Cu at (148.0, 120.0)
- added TP6: Buck_OUT_3.3V, TestPoint:TestPoint_Pad_1.0x1.0mm, F.Cu at (146.5, 110.5)
- added TP7: ESP32_BOOT, TestPoint:TestPoint_Pad_1.0x1.0mm, F.Cu at (119.5, 124.5)
- added TP8: I2C_SDA, TestPoint:TestPoint_Pad_1.0x1.0mm, F.Cu at (135.0, 157.5)
- added TP9: I2C_SCL, TestPoint:TestPoint_Pad_1.0x1.0mm, F.Cu at (139.5, 143.0)
- added U11: Display, Cube_OS_Footprint:CON_5034801200_MOL, F.Cu at (126.5, 114.2)
- added U4: LDLN025J28R, Cube_OS_Footprint:FLIPCHIP4_0P658X0P658_STM, F.Cu at (142.3, 132.8)
- R6: value 2.4 kΩ -> 3.9kΩ
- U1: value ESP32-S3-WROOM-1-N8R8 -> ESP32-S3-WROOM-1-N8R2
- U10, U12, U9: footprint Cube_OS_Footprint:CONN_FH35C-15S-0.3SHW50_HIR -> Cube_OS_Footprint:CON_5034801200_MOL
- U7: value Top Display -> TCA6408ARGTR; footprint Cube_OS_Footprint:CONN_FH35C-15S-0.3SHW50_HIR -> Cube_OS_Footprint:RGT16_1P45X1P45
- moved SW1 60.2 mm to (152.0, 155.5)
- moved M1 56.0 mm to (153.0, 135.7)
- moved J1 46.3 mm to (156.0, 151.0)
- moved SW2 44.8 mm to (142.2, 149.8)
- moved R16 40.5 mm to (146.5, 153.0)
- moved TH1 30.4 mm to (156.2, 141.8), turned to 90 degrees
- moved U7 22.8 mm to (141.5, 120.8), turned to 180 degrees
- moved U5 5.14 mm to (131.2, 156.2)
- moved R12 0.31 mm to (151.7, 113.0), turned to 180 degrees
- turned U10 to 90 degrees
- turned U12 to 0 degrees
- turned U9 to 180 degrees
Connections:
- C2 pad 1: Net-(U14-EN) -> Net-(U14-VIN)
- J1 pad 1: Net-(J1-Pin_1) -> GND
- J1 pad 2: GND -> +BAT
- R12 pad 1: Net-(U1-IO39) -> 3.3V
- R13 pad 1: Net-(U1-IO38) -> 3.3V
- R16 pad 2: Net-(U1-IO5) -> Net-(U7-P2)
- SW1 pad 2: Net-(J1-Pin_1) -> Net-(U14-EN)
- SW1 pad 5: +BAT -> Net-(U14-VIN)
- U1 pad 10: /IMU_INT1 -> /CAM_HREF
- U1 pad 15: /CAM_HREF -> unconnected-(U1-IO3-Pad15)
- U1 pad 16: /CAM_D6 -> unconnected-(U1-IO46-Pad16)
- U1 pad 26: /CAM_D5 -> unconnected-(U1-IO45-Pad26)
- U1 pad 27: /CAM_VSYNC -> Net-(U1-IO0)
- U1 pad 3: 3.3V -> Net-(U1-EN)
- U1 pad 31: Net-(U1-IO38) -> /CAM_D6
- U1 pad 32: Net-(U1-IO39) -> /CAM_D5
- U1 pad 5: Net-(U1-IO5) -> /CAM_VSYNC
- U10 pad 1: 3.3V -> LEDK
- U10 pad 10: /DISP_DC -> 3.3V
- U10 pad 11: /DISP_MOSI -> /DISP_RIGHT_CS
- U10 pad 12: unconnected-(U10-TE-Pad12) -> GND
- U10 pad 2: LEDK -> Net-(U10-LEDA)
- U10 pad 3: 3.3V -> GND
- U10 pad 4: 3.3V -> unconnected-(U10-SDO-Pad4)
- U10 pad 5: GND -> /DISP_RST
- U10 pad 6: GND -> /DISP_MOSI
- U10 pad 7: /DISP_RST -> /DISP_DC
- U10 pad 8: /DISP_RIGHT_CS -> /DISP_SCLK
- U10 pad 9: /DISP_SCLK -> 3.3V
- U12 pad 1: 3.3V -> LEDK
- U12 pad 10: /DISP_DC -> 3.3V
- U12 pad 11: /DISP_MOSI -> /DISP_LEFT_CS
- U12 pad 12: unconnected-(U12-TE-Pad12) -> GND
- U12 pad 2: LEDK -> Net-(U12-LEDA)
- U12 pad 3: 3.3V -> GND
- U12 pad 4: 3.3V -> unconnected-(U12-SDO-Pad4)
- U12 pad 5: GND -> /DISP_RST
- U12 pad 6: GND -> /DISP_MOSI
- U12 pad 7: /DISP_RST -> /DISP_DC
- U12 pad 8: /DISP_LEFT_CS -> /DISP_SCLK
- U12 pad 9: /DISP_SCLK -> 3.3V
- U14 pad 10: Net-(U14-EN) -> Net-(U14-VIN)
- U2 pad 4: 3.3V -> GND
- U5 pad 4: /IMU_INT1 -> unconnected-(U5-INT1-Pad4)
- U7 pad 1: 3.3V -> Net-(U7-*RESET)
- U7 pad 10: /DISP_DC -> unconnected-(U7-P7-Pad10)
- U7 pad 11: /DISP_MOSI -> Net-(U7-*INT)
- U7 pad 12: unconnected-(U7-TE-Pad12) -> /I2C_SCL
- U7 pad 13: GND -> /I2C_SDA
- U7 pad 14: GND -> 3.3V
- U7 pad 15: GND -> 3.3V
- U7 pad 2: LEDK -> /CHG_PGOOD
- U7 pad 3: 3.3V -> /CHG_STAT
- U7 pad 4: 3.3V -> Net-(U7-P2)
- U7 pad 5: GND -> unconnected-(U7-P3-Pad5)
- U7 pad 7: /DISP_RST -> unconnected-(U7-P4-Pad7)
- U7 pad 8: /DISP_TOP_CS -> unconnected-(U7-P5-Pad8)
- U7 pad 9: /DISP_SCLK -> unconnected-(U7-P6-Pad9)
- U8 pad 10: Net-(U14-EN) -> Net-(U14-VIN)
- U8 pad 11: Net-(U14-EN) -> Net-(U14-VIN)
- U9 pad 1: 3.3V -> LEDK
- U9 pad 10: /DISP_DC -> 3.3V
- U9 pad 11: /DISP_MOSI -> /DISP_FRONT_CS
- U9 pad 12: unconnected-(U9-TE-Pad12) -> GND
- U9 pad 2: LEDK -> Net-(U9-LEDA)
- U9 pad 3: 3.3V -> GND
- U9 pad 4: 3.3V -> unconnected-(U9-SDO-Pad4)
- U9 pad 5: GND -> /DISP_RST
- U9 pad 6: GND -> /DISP_MOSI
- U9 pad 7: /DISP_RST -> /DISP_DC
- U9 pad 8: /DISP_FRONT_CS -> /DISP_SCLK
- U9 pad 9: /DISP_SCLK -> 3.3V
Routing:
- net Net-(U1-IO5): track 85.0 -> 0.00 mm, vias 2 -> 0
- net Net-(U1-EN): track 0.00 -> 79.2 mm, vias 0 -> 3
- net Net-(U14-VIN): track 0.00 -> 65.1 mm, vias 0 -> 4
- net /CAM_VSYNC: track 12.8 -> 66.3 mm
- net /SERVO1_PWM: track 29.5 -> 79.2 mm, vias 2 -> 4
- net Net-(U7-P2): track 0.00 -> 49.0 mm, vias 0 -> 2
- net Net-(U1-IO0): track 0.00 -> 48.7 mm, vias 0 -> 4
- net Net-(U14-EN): track 9.55 -> 54.2 mm
- net Net-(U1-IO39): track 41.0 -> 0.00 mm, vias 4 -> 0
- net Net-(U1-IO38): track 39.6 -> 0.00 mm, vias 4 -> 0
- net GND: track 103.7 -> 142.6 mm, vias 63 -> 59
- net /CHG_PGOOD: track 2.26 -> 39.0 mm, vias 0 -> 6
- net Net-(U8-TS): track 5.92 -> 36.2 mm
- net Net-(J1-Pin_1): track 29.9 -> 0.00 mm
- net /I2C_SCL: track 44.2 -> 73.5 mm, vias 5 -> 7
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- added copper zone on F.Cu, net (none)
Other:
- outline, holes or cut-outs redrawn
- board text added: "+BAT"
- board text added: "GND"
