File: PCB/Rev A/source/Cube OS/Cube OS.kicad_pcb (KiCad board)
At the start: 4 copper layers, 60 x 60 mm, 81 parts, among them J1 1S 3.7 V LiPo, J2 KH-TYPE-C-16P, M1 Motor_Servo, M2 Motor_Servo, Q1 AO3400A, SW1 JS202011JAQN, SW2 SPPJ320600, SW3 RESET, SW4 BOOT, U1 ESP32-S3-WROOM-1-N8R2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

Commit message: Update Rev A PCB production package
Routing:
- net GND: vias 59 -> 193

Commit message: Update project assets and LFS tracking
Parts:
- added R25: 100kΩ, Resistor_SMD:R_0402_1005Metric, F.Cu at (150.0, 152.5)
Routing:
- net Net-(U14-EN): track 54.2 -> 55.7 mm
- net GND: vias 193 -> 194
