File: PCB/Rev A/source/Cube OS/Cube OS.kicad_sch (KiCad schematic)
At the start: 81 parts, among them J1 1S 3.7 V LiPo, J2 KH-TYPE-C-16P, M1 Motor_Servo, M2 Motor_Servo, Q1 AO3400A, SW1 JS202011JAQN, SW2 SPPJ320600, SW3 RESET, SW4 BOOT, U1 ESP32-S3-WROOM-1-N8R2, U10 Right Display, U11 Display, U12 Left Display, U13 MAX98357AETE+T, U14 TPS63802DLAR, U16 TPS7A0212PDBVR, U2 SHT45-AD1B-R2_Temp_Hu, U3 VEML7700-TT_SHORT, U4 LDLN025J28R, U5 ISM330DHCXTR_GYRO, U7 TCA6408ARGTR, U8 BQ24074RGTR_Batt, U9 Front Display

Commit message: Revert "Update Rev A PCB production package"
This reverts commit 683648053a19518fab4d864910172dd1a356c20e.
Parts:
- removed C10: 4.7uF, Capacitor_SMD:C_0402_1005Metric, symbol Device:C
- removed C11: 47uF, Capacitor_SMD:C_0805_2012Metric, symbol Device:C
- removed C7, C8, C9: 1 uF, Capacitor_SMD:C_0402_1005Metric, symbol Device:C
- removed R15, R20, R21, R22, R24: 10 kΩ, Resistor_SMD:R_0402_1005Metric, symbol Device:R
- removed R17, R18, R19, R23: 10Ω, Resistor_SMD:R_0603_1608Metric, symbol Device:R
- removed SW3: RESET, Cube_OS_Footprint:SW_TS-1088_XNP, symbol Switch:SW_Push
- removed SW4: BOOT, Cube_OS_Footprint:SW_TS-1088_XNP, symbol Switch:SW_Push
- removed TP1: GND, TestPoint:TestPoint_Pad_1.0x1.0mm, symbol Connector:TestPoint
- removed TP10: CHG_PGOOD, TestPoint:TestPoint_Pad_1.0x1.0mm, symbol Connector:TestPoint
- removed TP11: CHG_STAT, TestPoint:TestPoint_Pad_1.0x1.0mm, symbol Connector:TestPoint
- removed TP12: DISP_SCLK, TestPoint:TestPoint_Pad_1.0x1.0mm, symbol Connector:TestPoint
- removed TP13: DISP_MOSI, TestPoint:TestPoint_Pad_1.0x1.0mm, symbol Connector:TestPoint
- removed TP14: DISP_BL_PWM, TestPoint:TestPoint_Pad_1.0x1.0mm, symbol Connector:TestPoint
- removed TP2: USB_VBUS, TestPoint:TestPoint_Pad_1.0x1.0mm, symbol Connector:TestPoint
- removed TP3: BAT_IN, TestPoint:TestPoint_Pad_1.0x1.0mm, symbol Connector:TestPoint
- removed TP4: ESP32_EN, TestPoint:TestPoint_Pad_1.0x1.0mm, symbol Connector:TestPoint
- removed TP5: Buck_IN, TestPoint:TestPoint_Pad_1.0x1.0mm, symbol Connector:TestPoint
- removed TP6: Buck_OUT_3.3V, TestPoint:TestPoint_Pad_1.0x1.0mm, symbol Connector:TestPoint
- removed TP7: ESP32_BOOT, TestPoint:TestPoint_Pad_1.0x1.0mm, symbol Connector:TestPoint
- removed TP8: I2C_SDA, TestPoint:TestPoint_Pad_1.0x1.0mm, symbol Connector:TestPoint
- removed TP9: I2C_SCL, TestPoint:TestPoint_Pad_1.0x1.0mm, symbol Connector:TestPoint
- removed U11: Display, Cube_OS_Footprint:CON_5034801200_MOL, symbol Cube_OS_Library:1.54{dblquote} IPS TFT LCD Display 240x240
- removed U4: LDLN025J28R, Cube_OS_Footprint:FLIPCHIP4_0P658X0P658_STM, symbol Cube_OS_Library:LDLN025J28R
- removed U7: TCA6408ARGTR, RGT16_1P45X1P45, symbol Cube_OS_Library:TCA6408ARGTR
- added U15: LDLN025M25R, Cube_OS_Footprint:SOT23_DBV_TEX, symbol Cube_OS_Library:LDLN025M25R
- added U7: Top Display, Cube_OS_Footprint:CONN_FH35C-15S-0.3SHW50_HIR, symbol Cube_OS_Library:1.54{dblquote} IPS TFT LCD Display 240x240
- R6: value 3.9kΩ -> 2.4 kΩ; JLCPCB C23018 -> C22940
- U1: value ESP32-S3-WROOM-1-N8R2 -> ESP32-S3-WROOM-1-N8R8; JLCPCB C2913204 -> C2913201
- U10, U12, U9: footprint Cube_OS_Footprint:CON_5034801200_MOL -> Cube_OS_Footprint:CONN_FH35C-15S-0.3SHW50_HIR; JLCPCB C587969 -> C2889267
Connections:
- net +BAT: now also SW1.5; no longer J1.2 (Pin_2)
- net 3.3V: now also U1.3 (EN), U10.1 (LEDA), U10.3 (VDD), U10.4 (VDDIO), U12.1 (LEDA), U12.3 (VDD), U12.4 (VDDIO), U2.4 (VSS), U9.1 (LEDA), U9.3 (VDD), U9.4 (VDDIO), U15.1 (VIN), U15.4 (EN), U7.1 (LEDA), U7.3 (VDD), U7.4 (VDDIO); no longer R12.1, R13.1, U10.10 (IOVCC), U10.9 (VCC), U12.10 (IOVCC), U12.9 (VCC), U9.10 (IOVCC), U9.9 (VCC)
- net CAM_D5: now also U1.26 (IO45); no longer U1.32 (IO39)
- net CAM_D6: now also U1.16 (IO46); no longer U1.31 (IO38)
- net CAM_HREF: now also U1.15 (IO3); no longer U1.10 (IO17)
- net CAM_VSYNC: now also U1.27 (IO0); no longer U1.5 (IO5)
- net DISP_DC: now also U10.10 (D/C), U12.10 (D/C), U9.10 (D/C), U7.10 (D/C); no longer U10.7 (D/C), U12.7 (D/C), U9.7 (D/C)
- net DISP_FRONT_CS: now also U9.8 (CS); no longer U9.11 (CS)
- net DISP_LEFT_CS: now also U12.8 (CS); no longer U12.11 (CS)
- net DISP_MOSI: now also U10.11 (SDA), U12.11 (SDA), U9.11 (SDA), U7.11 (SDA); no longer U10.6 (SDA), U12.6 (SDA), U9.6 (SDA)
- net DISP_RIGHT_CS: now also U10.8 (CS); no longer U10.11 (CS)
- net DISP_RST: now also U10.7 (RESET), U12.7 (RESET), U9.7 (RESET), U7.7 (RESET); no longer U10.5 (RESET), U12.5 (RESET), U9.5 (RESET)
- net DISP_SCLK: now also U10.9 (SCLK), U12.9 (SCLK), U9.9 (SCLK), U7.9 (SCLK); no longer U10.8 (SCL), U12.8 (SCL), U9.8 (SCL)
- net DISP_TOP_CS: now also U7.8 (CS)
- net GND: now also J1.2 (Pin_2), U10.13 (GND), U10.14 (GND), U10.15 (GND), U10.16 (GND), U10.17 (GND), U10.5 (GND), U10.6 (GND), U12.13 (GND), U12.14 (GND), U12.15 (GND), U12.16 (GND), U12.17 (GND), U12.5 (GND), U12.6 (GND), U9.13 (GND), U9.14 (GND), U9.15 (GND), U9.16 (GND), U9.17 (GND), U9.5 (GND), U9.6 (GND), U15.3 (GND), U7.13 (GND), U7.14 (GND), U7.15 (GND), U7.16 (GND), U7.17 (GND), U7.5 (GND), U7.6 (GND); no longer J1.1 (Pin_1), U10.12 (GND), U10.3 (GND), U10.P1, U10.P2, U12.12 (GND), U12.3 (GND), U12.P1, U12.P2, U2.4 (VSS), U9.12 (GND), U9.3 (GND), U9.P1, U9.P2
- net LEDK: now also U10.2 (LEDK), U12.2 (LEDK), U9.2 (LEDK), U7.2 (LEDK); no longer U10.1 (LEDK), U12.1 (LEDK), U9.1 (LEDK)
- net at CAM1.4 (AVDD): now also U15.2 (VOUT)
- net at C2.1, U14.10 (VIN), U8.10 (OUT)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: now also U14.1 (EN); no longer SW1.5
- net at SW1.2: now also J1.1 (Pin_1); no longer U14.1 (EN)
- net IMU_INT1: now reaches U5.4 (INT1)
- net IMU_INT1: now also U1.10 (IO17)
- net at R16.2: now also U1.5 (IO5)
- new net: R12.1, U1.32 (IO39)
- new net: R13.1, U1.31 (IO38)
- no-connect marks 25 -> 17
Other:
- moved on the sheet: R12, R13, R16, SW1, SW2

Commit message: Update Rev A PCB production package
Parts:
- removed U15: LDLN025M25R, Cube_OS_Footprint:SOT23_DBV_TEX, symbol Cube_OS_Library:LDLN025M25R
- removed U7: Top Display, Cube_OS_Footprint:CONN_FH35C-15S-0.3SHW50_HIR, symbol Cube_OS_Library:1.54{dblquote} IPS TFT LCD Display 240x240
- added C10: 4.7uF, Capacitor_SMD:C_0402_1005Metric, symbol Device:C
- added C11: 47uF, Capacitor_SMD:C_0805_2012Metric, symbol Device:C
- added C7, C8, C9: 1 uF, Capacitor_SMD:C_0402_1005Metric, symbol Device:C
- added R15, R20, R21, R22, R24: 10 kΩ, Resistor_SMD:R_0402_1005Metric, symbol Device:R
- added R17, R18, R19, R23: 10Ω, Resistor_SMD:R_0603_1608Metric, symbol Device:R
- added SW3: RESET, Cube_OS_Footprint:SW_TS-1088_XNP, symbol Switch:SW_Push
- added SW4: BOOT, Cube_OS_Footprint:SW_TS-1088_XNP, symbol Switch:SW_Push
- added TP1: GND, TestPoint:TestPoint_Pad_1.0x1.0mm, symbol Connector:TestPoint
- added TP10: CHG_PGOOD, TestPoint:TestPoint_Pad_1.0x1.0mm, symbol Connector:TestPoint
- added TP11: CHG_STAT, TestPoint:TestPoint_Pad_1.0x1.0mm, symbol Connector:TestPoint
- added TP12: DISP_SCLK, TestPoint:TestPoint_Pad_1.0x1.0mm, symbol Connector:TestPoint
- added TP13: DISP_MOSI, TestPoint:TestPoint_Pad_1.0x1.0mm, symbol Connector:TestPoint
- added TP14: DISP_BL_PWM, TestPoint:TestPoint_Pad_1.0x1.0mm, symbol Connector:TestPoint
- added TP2: USB_VBUS, TestPoint:TestPoint_Pad_1.0x1.0mm, symbol Connector:TestPoint
- added TP3: BAT_IN, TestPoint:TestPoint_Pad_1.0x1.0mm, symbol Connector:TestPoint
- added TP4: ESP32_EN, TestPoint:TestPoint_Pad_1.0x1.0mm, symbol Connector:TestPoint
- added TP5: Buck_IN, TestPoint:TestPoint_Pad_1.0x1.0mm, symbol Connector:TestPoint
- added TP6: Buck_OUT_3.3V, TestPoint:TestPoint_Pad_1.0x1.0mm, symbol Connector:TestPoint
- added TP7: ESP32_BOOT, TestPoint:TestPoint_Pad_1.0x1.0mm, symbol Connector:TestPoint
- added TP8: I2C_SDA, TestPoint:TestPoint_Pad_1.0x1.0mm, symbol Connector:TestPoint
- added TP9: I2C_SCL, TestPoint:TestPoint_Pad_1.0x1.0mm, symbol Connector:TestPoint
- added U11: Display, Cube_OS_Footprint:CON_5034801200_MOL, symbol Cube_OS_Library:1.54{dblquote} IPS TFT LCD Display 240x240
- added U4: LDLN025J28R, Cube_OS_Footprint:FLIPCHIP4_0P658X0P658_STM, symbol Cube_OS_Library:LDLN025J28R
- added U7: TCA6408ARGTR, RGT16_1P45X1P45, symbol Cube_OS_Library:TCA6408ARGTR
- R6: value 2.4 kΩ -> 3.9kΩ; JLCPCB C22940 -> C23018
- U1: value ESP32-S3-WROOM-1-N8R8 -> ESP32-S3-WROOM-1-N8R2; JLCPCB C2913201 -> C2913204
- U10, U12, U9: footprint Cube_OS_Footprint:CONN_FH35C-15S-0.3SHW50_HIR -> Cube_OS_Footprint:CON_5034801200_MOL; JLCPCB C2889267 -> C587969
Connections:
- net +BAT: now also J1.2 (Pin_2), C10.1, C11.1, TP3.1; no longer SW1.5
- net 3.3V: now also R12.1, R13.1, U10.10 (IOVCC), U10.9 (VCC), U12.10 (IOVCC), U12.9 (VCC), U9.10 (IOVCC), U9.9 (VCC), C8.1, R15.1, R17.2, R18.2, R19.2, R20.1, R21.2, R23.2, R24.2, TP6.1, U11.10 (IOVCC), U11.9 (VCC), U4.A1 (VIN), U4.B1 (EN), U7.14 (VCCP), U7.15 (VCCI); no longer U1.3 (EN), U10.1 (LEDA), U10.3 (VDD), U10.4 (VDDIO), U12.1 (LEDA), U12.3 (VDD), U12.4 (VDDIO), U2.4 (VSS), U9.1 (LEDA), U9.3 (VDD), U9.4 (VDDIO)
- net CAM_D5: now also U1.32 (IO39); no longer U1.26 (IO45)
- net CAM_D6: now also U1.31 (IO38); no longer U1.16 (IO46)
- net CAM_HREF: now also U1.10 (IO17); no longer U1.15 (IO3)
- net CAM_VSYNC: now also U1.5 (IO5); no longer U1.27 (IO0)
- net CHG_PGOOD: now also TP10.1, U7.2 (P0)
- net CHG_STAT: now also TP11.1, U7.3 (P1)
- net DISP_BL_PWM: now also TP14.1
- net DISP_DC: now also U10.7 (D/C), U12.7 (D/C), U9.7 (D/C), U11.7 (D/C); no longer U10.10 (D/C), U12.10 (D/C), U9.10 (D/C)
- net DISP_FRONT_CS: now also U9.11 (CS); no longer U9.8 (CS)
- net DISP_LEFT_CS: now also U12.11 (CS); no longer U12.8 (CS)
- net DISP_MOSI: now also U10.6 (SDA), U12.6 (SDA), U9.6 (SDA), TP13.1, U11.6 (SDA); no longer U10.11 (SDA), U12.11 (SDA), U9.11 (SDA)
- net DISP_RIGHT_CS: now also U10.11 (CS); no longer U10.8 (CS)
- net DISP_RST: now also U10.5 (RESET), U12.5 (RESET), U9.5 (RESET), U11.5 (RESET); no longer U10.7 (RESET), U12.7 (RESET), U9.7 (RESET)
- net DISP_SCLK: now also U10.8 (SCL), U12.8 (SCL), U9.8 (SCL), TP12.1, U11.8 (SCL); no longer U10.9 (SCLK), U12.9 (SCLK), U9.9 (SCLK)
- net DISP_TOP_CS: now also U11.11 (CS)
- net GND: now also J1.1 (Pin_1), U10.12 (GND), U10.3 (GND), U10.P1, U10.P2, U12.12 (GND), U12.3 (GND), U12.P1, U12.P2, U2.4 (VSS), U9.12 (GND), U9.3 (GND), U9.P1, U9.P2, C10.2, C11.2, C7.2, C8.2, C9.2, R22.2, SW3.1, SW4.1, TP1.1, U11.12 (GND), U11.3 (GND), U11.P1, U11.P2, U4.B2 (GND), U7.16 (ADDR), U7.17 (EPAD), U7.6 (GND); no longer J1.2 (Pin_2), U10.13 (GND), U10.14 (GND), U10.15 (GND), U10.16 (GND), U10.17 (GND), U10.5 (GND), U10.6 (GND), U12.13 (GND), U12.14 (GND), U12.15 (GND), U12.16 (GND), U12.17 (GND), U12.5 (GND), U12.6 (GND), U9.13 (GND), U9.14 (GND), U9.15 (GND), U9.16 (GND), U9.17 (GND), U9.5 (GND), U9.6 (GND)
- net I2C_SCL: now also TP9.1, U7.12 (SCL)
- net I2C_SDA: now also TP8.1, U7.13 (SDA)
- net I2S_MIC_DATA: now also R22.1
- net LEDK: now also U10.1 (LEDK), U12.1 (LEDK), U9.1 (LEDK), U11.1 (LEDK); no longer U10.2 (LEDK), U12.2 (LEDK), U9.2 (LEDK)
- net USB_VBUS: now also TP2.1
- net at C2.1, U14.10 (VIN), U8.10 (OUT)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: now also SW1.5, TP5.1; no longer U14.1 (EN)
- net at CAM1.4 (AVDD): now also C9.1, U4.A2 (VOUT)
- net at SW1.2: now also U14.1 (EN); no longer J1.1 (Pin_1)
- net at CAM1.10 (DVDD), U16.5 (OUT): now also C7.1
- net at R16.2: now also U7.4 (P2); no longer U1.5 (IO5)
- net IMU_INT1: no longer names the net of U5.4 (INT1)
- net IMU_INT1: no longer U1.10 (IO17)
- new net: R20.2, U7.11 (*INT)
- new net: R19.1, U10.2 (LEDA)
- new net: R17.1, U9.2 (LEDA)
- new net: R21.1, U7.1 (*RESET)
- new net: R18.1, U12.2 (LEDA)
- new net: R15.2, SW3.2, TP4.1, U1.3 (EN)
- new net: R24.1, SW4.2, TP7.1, U1.27 (IO0)
- new net: R23.1, U11.2 (LEDA)
- no-connect marks 17 -> 25
Other:
- moved on the sheet: R12, R13, R16, SW1, SW2

Commit message: Update project assets and LFS tracking
Parts:
- added R25: 100kΩ, Resistor_SMD:R_0402_1005Metric, symbol Device:R
- U7: footprint RGT16_1P45X1P45 -> Cube_OS_Footprint:RGT16_1P45X1P45
Connections:
- net GND: now also R25.2
- net at SW1.2, U14.1 (EN): now also R25.1
Changed lines of the file:
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@@
 	(wire
 		(pts
+			(xy 182.88 215.9) (xy 182.88 217.17)
+		)
+		(stroke
+			(width 0)
+			(type default)
+		)
+	)
+	(wire
+		(pts
 			(xy 115.57 201.93) (xy 115.57 215.9)
 		)
@@
 	(wire
 		(pts
+			(xy 184.15 208.28) (xy 184.15 207.01)
+		)
+		(stroke
+			(width 0)
+			(type default)
+		)
+	)
+	(wire
+		(pts
 			(xy 39.37 116.84) (xy 39.37 161.29)
 		)
@@
 	(wire
 		(pts
+			(xy 182.88 208.28) (xy 184.15 208.28)
+		)
+		(stroke
+			(width 0)
+			(type default)
+		)
+	)
+	(wire
+		(pts
 			(xy 25.4 124.46) (xy 36.83 124.46)
 		)
@@
 	)
 	(symbol
+		(lib_id "power:GND")
+		(at 182.88 217.17 0)
+		(unit 1)
+		(exclude_from_sim no)
+		(in_bom yes)
+		(on_board yes)
+		(dnp no)
+		(fields_autoplaced yes)
+		(property "Reference" "#PWR054"
+			(at 182.88 223.52 0)
+			(effects
+				(font
+					(size 1.27 1.27)
+				)
+				(hide yes)
+			)
+		)
+		(property "Value" "GND"
+			(at 182.88 222.25 0)
+			(effects
+				(font
+					(size 1.27 1.27)
+				)
+				(hide yes)
+			)
+		)
+		(property "Footprint" ""
+			(at 182.88 217.17 0)
+			(effects
+				(font
+					(size 1.27 1.27)
+				)
+				(hide yes)
+			)
+		)
+		(property "Datasheet" ""
+			(at 182.88 217.17 0)
+			(effects
+				(font
+					(size 1.27 1.27)
+				)
+				(hide yes)
+			)
+		)
+		(property "Description" "Power symbol creates a global label with name \"GND\" , ground"
+			(at 182.88 217.17 0)
+			(effects
+				(font
+					(size 1.27 1.27)
+				)
+				(hide yes)
+			)
+		)
+		(pin "1"
+		)
+		(instances
+			(project "Cube OS"
+				(path "/1824f342-0d29-49b4-8da8-99a2a0b66501"
+					(reference "#PWR054")
+					(unit 1)
+				)
+			)
+		)
+	)
+	(symbol
 		(lib_id "Cube_OS_Library:JS202011JAQN")
 		(at 179.07 170.18 90)
@@
 	(symbol
 		(lib_id "Device:R")
+		(at 182.88 212.09 0)
+		(unit 1)
+		(exclude_from_sim no)
+		(in_bom yes)
+		(on_board yes)
+		(dnp no)
+		(fields_autoplaced yes)
+		(property "Reference" "R25"
+			(at 185.42 210.8199 0)
+			(effects
+				(font
+					(size 1.27 1.27)
+				)
+				(justify left)
+			)
+		)
+		(property "Value" "100kΩ"
+			(at 185.42 213.3599 0)
+			(effects
+				(font
+					(size 1.27 1.27)
+				)
+				(justify left)
+			)
+		)
+		(property "Footprint" "Resistor_SMD:R_0402_1005Metric"
+			(at 181.102 212.09 90)
+			(effects
+				(font
+					(size 1.27 1.27)
+				)
+				(hide yes)
+			)
+		)
+		(property "Datasheet" "~"
+			(at 182.88 212.09 0)
+			(effects
+				(font
+					(size 1.27 1.27)
+				)
+				(hide yes)
+			)
+		)
+		(property "Description" "Resistor"
+			(at 182.88 212.09 0)
+			(effects
+				(font
+					(size 1.27 1.27)
+				)
+				(hide yes)
+			)
+		)
+		(property "JLCPCB" "C25741"
+			(at 182.88 212.09 0)
+			(effects
+				(font
+					(size 1.27 1.27)
+				)
+				(hide yes)
+			)
+		)
+		(pin "1"
+		)
+		(pin "2"
+		)
+		(instances
+			(project "Cube OS"
+				(path "/1824f342-0d29-49b4-8da8-99a2a0b66501"
+					(reference "R25")
+					(unit 1)
+				)
+			)
+		)
+	)
+	(symbol
+		(lib_id "Device:R")
 		(at 83.82 73.66 90)
 		(unit 1)
@@
 		(pin "4"
 		)
-		(pin "MT1"
-		)
 		(pin "15"
 		)
-		(pin "MT2"
-		)
 		(pin "2"
 		)
@@
 			)
 		)
-		(property "Footprint" "RGT16_1P45X1P45"
+		(property "Footprint" "Cube_OS_Footprint:RGT16_1P45X1P45"
 			(at 120.65 220.98 0)
 			(effects
